File: hardware/capelets/solar/capelet_solar.sch (EAGLE design)
At the start: 4 parts

Commit message: hardware: fancy frames around capelet schematics
Parts:
- ROC1: value (none) -> 8M
- ROC2: value (none) -> 2M
Other:
- moved on the sheet: ROC1, ROC2, X1-1, X1-2
Changed lines of the file:
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@@
 <?xml version="1.0" encoding="utf-8"?>
 <!DOCTYPE eagle SYSTEM "eagle.dtd">
-<eagle version="9.3.2">
+<eagle version="9.4.2">
 <drawing>
 <settings>
@@
 </classes>
 <parts>
-<part name="ROC2" library="mylib" deviceset="R_SMD" device="0805"/>
-<part name="ROC1" library="mylib" deviceset="R_SMD" device="0805"/>
+<part name="ROC2" library="mylib" deviceset="R_SMD" device="0805" value="2M"/>
+<part name="ROC1" library="mylib" deviceset="R_SMD" device="0805" value="8M"/>
 <part name="GND1" library="supply1" library_urn="urn:adsk.eagle:library:371" deviceset="GND" device=""/>
 <part name="U$1" library="shepherd" deviceset="SHPRD_CPLT_H" device=""/>
 <part name="X1" library="con-wago-500" library_urn="urn:adsk.eagle:library:195" deviceset="W237-102" device="" package3d_urn="urn:adsk.eagle:package:10688/1"/>
+<part name="FRAME1" library="frames" library_urn="urn:adsk.eagle:library:229" deviceset="A4L-LOC" device=""/>
 </parts>
 <sheets>
@@
 </plain>
 <instances>
-<instance part="ROC2" gate="G$1" x="-17.78" y="-2.54" smashed="yes" rot="R90">
-<attribute name="NAME" x="-19.2786" y="-6.35" size="1.778" layer="95" rot="R90"/>
-<attribute name="VALUE" x="-14.478" y="-6.35" size="1.778" layer="96" rot="R90"/>
-</instance>
-<instance part="ROC1" gate="G$1" x="-17.78" y="-17.78" smashed="yes" rot="R90">
-<attribute name="NAME" x="-19.2786" y="-21.59" size="1.778" layer="95" rot="R90"/>
-<attribute name="VALUE" x="-14.478" y="-21.59" size="1.778" layer="96" rot="R90"/>
-</instance>
-<instance part="GND1" gate="1" x="-17.78" y="-33.02" smashed="yes">
-<attribute name="VALUE" x="-20.32" y="-35.56" size="1.778" layer="96"/>
-</instance>
-<instance part="U$1" gate="G$1" x="2.54" y="0" smashed="yes"/>
-<instance part="U$1" gate="G$2" x="119.38" y="-68.58" smashed="yes"/>
-<instance part="U$1" gate="G$3" x="177.8" y="-68.58" smashed="yes"/>
-<instance part="X1" gate="-1" x="-45.72" y="5.08" smashed="yes">
-<attribute name="NAME" x="-45.72" y="5.969" size="1.778" layer="95" rot="R180"/>
-</instance>
-<instance part="X1" gate="-2" x="-45.72" y="0" smashed="yes">
-<attribute name="VALUE" x="-48.26" y="-3.683" size="1.778" layer="96"/>
-<attribute name="NAME" x="-45.72" y="0.889" size="1.778" layer="95" rot="R180"/>
+<instance part="ROC2" gate="G$1" x="50.8" y="53.34" smashed="yes" rot="R90">
+<attribute name="NAME" x="49.3014" y="49.53" size="1.778" layer="95" rot="R90"/>
+<attribute name="VALUE" x="54.102" y="49.53" size="1.778" layer="96" rot="R90"/>
+</instance>
+<instance part="ROC1" gate="G$1" x="50.8" y="38.1" smashed="yes" rot="R90">
+<attribute name="NAME" x="49.3014" y="34.29" size="1.778" layer="95" rot="R90"/>
+<attribute name="VALUE" x="54.102" y="34.29" size="1.778" layer="96" rot="R90"/>
+</instance>
+<instance part="GND1" gate="1" x="50.8" y="22.86" smashed="yes">
+<attribute name="VALUE" x="48.26" y="20.32" size="1.778" layer="96"/>
+</instance>
+<instance part="U$1" gate="G$1" x="71.12" y="55.88" smashed="yes"/>
+<instance part="U$1" gate="G$2" x="106.68" y="78.74" smashed="yes"/>
+<instance part="U$1" gate="G$3" x="165.1" y="78.74" smashed="yes"/>
+<instance part="X1" gate="-1" x="22.86" y="60.96" smashed="yes">
+<attribute name="NAME" x="22.86" y="61.849" size="1.778" layer="95" rot="R180"/>
+</instance>
+<instance part="X1" gate="-2" x="22.86" y="55.88" smashed="yes">
+<attribute name="VALUE" x="20.32" y="52.197" size="1.778" layer="96"/>
+<attribute name="NAME" x="22.86" y="56.769" size="1.778" layer="95" rot="R180"/>
+</instance>
+<instance part="FRAME1" gate="G$1" x="0" y="0" smashed="yes">
+<attribute name="DRAWING_NAME" x="217.17" y="15.24" size="2.54" layer="94"/>
+<attribute name="LAST_DATE_TIME" x="217.17" y="10.16" size="2.286" layer="94"/>
+<attribute name="SHEET" x="230.505" y="5.08" size="2.54" layer="94"/>
 </instance>
 </instances>
@@
 <segment>
 <pinref part="ROC2" gate="G$1" pin="2"/>
-<wire x1="-17.78" y1="2.54" x2="-17.78" y2="5.08" width="0.1524" layer="91"/>
-<wire x1="-17.78" y1="5.08" x2="-2.54" y2="5.08" width="0.1524" layer="91"/>
+<wire x1="50.8" y1="58.42" x2="50.8" y2="60.96" width="0.1524" layer="91"/>
+<wire x1="50.8" y1="60.96" x2="66.04" y2="60.96" width="0.1524" layer="91"/>
 <pinref part="U$1" gate="G$1" pin="V_H"/>
-<wire x1="-17.78" y1="5.08" x2="-40.64" y2="5.08" width="0.1524" layer="91"/>
-<junction x="-17.78" y="5.08"/>
+<wire x1="50.8" y1="60.96" x2="27.94" y2="60.96" width="0.1524" layer="91"/>
+<junction x="50.8" y="60.96"/>
 <pinref part="X1" gate="-1" pin="KL"/>
 </segment>
@@
 <pinref part="ROC2" gate="G$1" pin="1"/>
 <pinref part="ROC1" gate="G$1" pin="2"/>
-<wire x1="-17.78" y1="-7.62" x2="-17.78" y2="-10.16" width="0.1524" layer="91"/>
-<wire x1="-17.78" y1="-10.16" x2="-17.78" y2="-12.7" width="0.1524" layer="91"/>
-<wire x1="-17.78" y1="-10.16" x2="-7.62" y2="-10.16" width="0.1524" layer="91"/>
-<wire x1="-7.62" y1="-10.16" x2="-7.62" y2="10.16" width="0.1524" layer="91"/>
-<junction x="-17.78" y="-10.16"/>
-<wire x1="-7.62" y1="10.16" x2="-2.54" y2="10.16" width="0.1524" layer="91"/>
+<wire x1="50.8" y1="48.26" x2="50.8" y2="45.72" width="0.1524" layer="91"/>
+<wire x1="50.8" y1="45.72" x2="50.8" y2="43.18" width="0.1524" layer="91"/>
+<wire x1="50.8" y1="45.72" x2="60.96" y2="45.72" width="0.1524" layer="91"/>
+<wire x1="60.96" y1="45.72" x2="60.96" y2="66.04" width="0.1524" layer="91"/>
+<junction x="50.8" y="45.72"/>
+<wire x1="60.96" y1="66.04" x2="66.04" y2="66.04" width="0.1524" layer="91"/>
 <pinref part="U$1" gate="G$1" pin="VOC_VD"/>
 </segment>
@@
 <pinref part="GND1" gate="1" pin="GND"/>
 <pinref part="ROC1" gate="G$1" pin="1"/>
-<wire x1="-17.78" y1="-30.48" x2="-17.78" y2="-25.4" width="0.1524" layer="91"/>
-<wire x1="-17.78" y1="-25.4" x2="-17.78" y2="-22.86" width="0.1524" layer="91"/>
-<wire x1="-38.1" y1="-25.4" x2="-17.78" y2="-25.4" width="0.1524" layer="91"/>
-<junction x="-17.78" y="-25.4"/>
-<wire x1="-17.78" y1="-25.4" x2="38.1" y2="-25.4" width="0.1524" layer="91"/>
-<wire x1="38.1" y1="-25.4" x2="38.1" y2="5.08" width="0.1524" layer="91"/>
-<wire x1="38.1" y1="5.08" x2="38.1" y2="10.16" width="0.1524" layer="91"/>
-<wire x1="33.02" y1="10.16" x2="38.1" y2="10.16" width="0.1524" layer="91"/>
-<wire x1="33.02" y1="5.08" x2="38.1" y2="5.08" width="0.1524" layer="91"/>
-<junction x="38.1" y="5.08"/>
+<wire x1="50.8" y1="25.4" x2="50.8" y2="30.48" width="0.1524" layer="91"/>
+<wire x1="50.8" y1="30.48" x2="50.8" y2="33.02" width="0.1524" layer="91"/>
+<wire x1="30.48" y1="30.48" x2="50.8" y2="30.48" width="0.1524" layer="91"/>
+<junction x="50.8" y="30.48"/>
+<wire x1="50.8" y1="30.48" x2="106.68" y2="30.48" width="0.1524" layer="91"/>
+<wire x1="106.68" y1="30.48" x2="106.68" y2="60.96" width="0.1524" layer="91"/>
+<wire x1="106.68" y1="60.96" x2="106.68" y2="66.04" width="0.1524" layer="91"/>
+<wire x1="101.6" y1="66.04" x2="106.68" y2="66.04" width="0.1524" layer="91"/>
+<wire x1="101.6" y1="60.96" x2="106.68" y2="60.96" width="0.1524" layer="91"/>
+<junction x="106.68" y="60.96"/>
 <pinref part="U$1" gate="G$1" pin="GND@1"/>
 <pinref part="U$1" gate="G$1" pin="GND@2"/>
-<wire x1="-40.64" y1="0" x2="-38.1" y2="0" width="0.1524" layer="91"/>
-<wire x1="-38.1" y1="0" x2="-38.1" y2="-25.4" width="0.1524" layer="91"/>
+<wire x1="27.94" y1="55.88" x2="30.48" y2="55.88" width="0.1524" layer="91"/>
+<wire x1="30.48" y1="55.88" x2="30.48" y2="30.48" width="0.1524" layer="91"/>
 <pinref part="X1" gate="-2" pin="KL"/>
 </segment>

Commit message: hardware: prepared capelets for external manufacturing
Parts:
- removed U$1: SHPRD_CPLT_H, shepherd:SHPRD_CPLT_H
- added P1: (no value), pinhead:PINHD-2X2
- added P8, P9: FE11-2, shepherd:FE11-2
Connections:
- removed net N$3: ROC1.2, ROC2.1, U$1G$1.VOC_VD
- new net N$5: P1.4, ROC1.2, ROC2.1
- net GND: now also P1.1, P1.2; no longer U$1G$1.GND@1, U$1G$1.GND@2
- net N$2: now also P1.3; no longer U$1G$1.V_H
Other:
- moved on the sheet: ROC1, ROC2, X1-1, X1-2
Changed lines of the file:
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@@
 <?xml version="1.0" encoding="utf-8"?>
 <!DOCTYPE eagle SYSTEM "eagle.dtd">
-<eagle version="9.4.2">
+<eagle version="9.5.2">
 <drawing>
 <settings>
@@
 <part name="ROC1" library="mylib" deviceset="R_SMD" device="0805" value="8M"/>
 <part name="GND1" library="supply1" library_urn="urn:adsk.eagle:library:371" deviceset="GND" device=""/>
-<part name="U$1" library="shepherd" deviceset="SHPRD_CPLT_H" device=""/>
 <part name="X1" library="con-wago-500" library_urn="urn:adsk.eagle:library:195" deviceset="W237-102" device="" package3d_urn="urn:adsk.eagle:package:10688/1"/>
 <part name="FRAME1" library="frames" library_urn="urn:adsk.eagle:library:229" deviceset="A4L-LOC" device=""/>
+<part name="P8" library="shepherd" deviceset="FE11-2" device=""/>
+<part name="P9" library="shepherd" deviceset="FE11-2" device=""/>
+<part name="P1" library="pinhead" library_urn="urn:adsk.eagle:library:325" deviceset="PINHD-2X2" device="" package3d_urn="urn:adsk.eagle:package:22455/2"/>
 </parts>
 <sheets>
@@
 </plain>
 <instances>
-<instance part="ROC2" gate="G$1" x="50.8" y="53.34" smashed="yes" rot="R90">
-<attribute name="NAME" x="49.3014" y="49.53" size="1.778" layer="95" rot="R90"/>
-<attribute name="VALUE" x="54.102" y="49.53" size="1.778" layer="96" rot="R90"/>
-</instance>
-<instance part="ROC1" gate="G$1" x="50.8" y="38.1" smashed="yes" rot="R90">
-<attribute name="NAME" x="49.3014" y="34.29" size="1.778" layer="95" rot="R90"/>
-<attribute name="VALUE" x="54.102" y="34.29" size="1.778" layer="96" rot="R90"/>
-</instance>
-<instance part="GND1" gate="1" x="50.8" y="22.86" smashed="yes">
-<attribute name="VALUE" x="48.26" y="20.32" size="1.778" layer="96"/>
-</instance>
-<instance part="U$1" gate="G$1" x="71.12" y="55.88" smashed="yes"/>
-<instance part="U$1" gate="G$2" x="106.68" y="78.74" smashed="yes"/>
-<instance part="U$1" gate="G$3" x="165.1" y="78.74" smashed="yes"/>
-<instance part="X1" gate="-1" x="22.86" y="60.96" smashed="yes">
-<attribute name="NAME" x="22.86" y="61.849" size="1.778" layer="95" rot="R180"/>
-</instance>
-<instance part="X1" gate="-2" x="22.86" y="55.88" smashed="yes">
-<attribute name="VALUE" x="20.32" y="52.197" size="1.778" layer="96"/>
-<attribute name="NAME" x="22.86" y="56.769" size="1.778" layer="95" rot="R180"/>
+<instance part="ROC2" gate="G$1" x="68.58" y="101.6" smashed="yes" rot="R90">
+<attribute name="NAME" x="67.0814" y="97.79" size="1.778" layer="95" rot="R90"/>
+<attribute name="VALUE" x="71.882" y="97.79" size="1.778" layer="96" rot="R90"/>
+</instance>
+<instance part="ROC1" gate="G$1" x="68.58" y="86.36" smashed="yes" rot="R90">
+<attribute name="NAME" x="67.0814" y="82.55" size="1.778" layer="95" rot="R90"/>
+<attribute name="VALUE" x="71.882" y="82.55" size="1.778" layer="96" rot="R90"/>
+</instance>
+<instance part="GND1" gate="1" x="68.58" y="71.12" smashed="yes">
+<attribute name="VALUE" x="66.04" y="68.58" size="1.778" layer="96"/>
+</instance>
+<instance part="X1" gate="-1" x="40.64" y="109.22" smashed="yes">
+<attribute name="NAME" x="40.64" y="110.109" size="1.778" layer="95" rot="R180"/>
+</instance>
+<instance part="X1" gate="-2" x="40.64" y="104.14" smashed="yes">
+<attribute name="VALUE" x="38.1" y="100.457" size="1.778" layer="96"/>
+<attribute name="NAME" x="40.64" y="105.029" size="1.778" layer="95" rot="R180"/>
 </instance>
 <instance part="FRAME1" gate="G$1" x="0" y="0" smashed="yes">
@@
 <attribute name="LAST_DATE_TIME" x="217.17" y="10.16" size="2.286" layer="94"/>
 <attribute name="SHEET" x="230.505" y="5.08" size="2.54" layer="94"/>
+</instance>
+<instance part="P8" gate="G$1" x="162.56" y="93.98" smashed="yes">
+<attribute name="NAME" x="156.21" y="111.76" size="1.778" layer="96"/>
+</instance>
+<instance part="P9" gate="G$1" x="200.66" y="93.98" smashed="yes">
+<attribute name="NAME" x="194.31" y="111.76" size="1.778" layer="96"/>
+</instance>
+<instance part="P1" gate="A" x="88.9" y="93.98" smashed="yes" rot="R180">
+<attribute name="NAME" x="97.79" y="88.265" size="1.778" layer="95" rot="R180"/>
+<attribute name="VALUE" x="97.79" y="99.06" size="1.778" layer="96" rot="R180"/>
 </instance>
 </instances>
@@
 <segment>
 <pinref part="ROC2" gate="G$1" pin="2"/>
-<wire x1="50.8" y1="58.42" x2="50.8" y2="60.96" width="0.1524" layer="91"/>
-<wire x1="50.8" y1="60.96" x2="66.04" y2="60.96" width="0.1524" layer="91"/>
-<pinref part="U$1" gate="G$1" pin="V_H"/>
-<wire x1="50.8" y1="60.96" x2="27.94" y2="60.96" width="0.1524" layer="91"/>
-<junction x="50.8" y="60.96"/>
+<wire x1="68.58" y1="106.68" x2="68.58" y2="109.22" width="0.1524" layer="91"/>
+<wire x1="68.58" y1="109.22" x2="45.72" y2="109.22" width="0.1524" layer="91"/>
 <pinref part="X1" gate="-1" pin="KL"/>
+<wire x1="68.58" y1="109.22" x2="99.06" y2="109.22" width="0.1524" layer="91"/>
+<junction x="68.58" y="109.22"/>
+<pinref part="P1" gate="A" pin="3"/>
+<wire x1="99.06" y1="109.22" x2="99.06" y2="93.98" width="0.1524" layer="91"/>
+<wire x1="99.06" y1="93.98" x2="93.98" y2="93.98" width="0.1524" layer="91"/>
 </segment>
 </net>
-<net name="N$3" class="0">
+<net name="N$5" class="0">
 <segment>
+<pinref part="ROC1" gate="G$1" pin="2"/>
 <pinref part="ROC2" gate="G$1" pin="1"/>
-<pinref part="ROC1" gate="G$1" pin="2"/>
-<wire x1="50.8" y1="48.26" x2="50.8" y2="45.72" width="0.1524" layer="91"/>
-<wire x1="50.8" y1="45.72" x2="50.8" y2="43.18" width="0.1524" layer="91"/>
-<wire x1="50.8" y1="45.72" x2="60.96" y2="45.72" width="0.1524" layer="91"/>
-<wire x1="60.96" y1="45.72" x2="60.96" y2="66.04" width="0.1524" layer="91"/>
-<junction x="50.8" y="45.72"/>
-<wire x1="60.96" y1="66.04" x2="66.04" y2="66.04" width="0.1524" layer="91"/>
-<pinref part="U$1" gate="G$1" pin="VOC_VD"/>
+<wire x1="68.58" y1="96.52" x2="68.58" y2="93.98" width="0.1524" layer="91"/>
+<pinref part="P1" gate="A" pin="4"/>
+<wire x1="68.58" y1="93.98" x2="68.58" y2="91.44" width="0.1524" layer="91"/>
+<wire x1="86.36" y1="93.98" x2="68.58" y2="93.98" width="0.1524" layer="91"/>
+<junction x="68.58" y="93.98"/>
 </segment>
 </net>
 <net name="GND" class="0">
 <segment>
+<pinref part="P1" gate="A" pin="2"/>
+<wire x1="86.36" y1="91.44" x2="81.28" y2="91.44" width="0.1524" layer="91"/>
+<pinref part="ROC1" gate="G$1" pin="1"/>
+<wire x1="68.58" y1="78.74" x2="68.58" y2="81.28" width="0.1524" layer="91"/>
+<wire x1="48.26" y1="78.74" x2="68.58" y2="78.74" width="0.1524" layer="91"/>
+<junction x="68.58" y="78.74"/>
+<wire x1="45.72" y1="104.14" x2="48.26" y2="104.14" width="0.1524" layer="91"/>
+<wire x1="48.26" y1="104.14" x2="48.26" y2="78.74" width="0.1524" layer="91"/>
+<pinref part="X1" gate="-2" pin="KL"/>
+<wire x1="81.28" y1="91.44" x2="81.28" y2="78.74" width="0.1524" layer="91"/>
+<wire x1="81.28" y1="78.74" x2="68.58" y2="78.74" width="0.1524" layer="91"/>
+<pinref part="P1" gate="A" pin="1"/>
+<wire x1="93.98" y1="91.44" x2="99.06" y2="91.44" width="0.1524" layer="91"/>
+<wire x1="99.06" y1="91.44" x2="99.06" y2="78.74" width="0.1524" layer="91"/>
+<wire x1="99.06" y1="78.74" x2="81.28" y2="78.74" width="0.1524" layer="91"/>
+<junction x="81.28" y="78.74"/>
 <pinref part="GND1" gate="1" pin="GND"/>
-<pinref part="ROC1" gate="G$1" pin="1"/>
-<wire x1="50.8" y1="25.4" x2="50.8" y2="30.48" width="0.1524" layer="91"/>
-<wire x1="50.8" y1="30.48" x2="50.8" y2="33.02" width="0.1524" layer="91"/>
-<wire x1="30.48" y1="30.48" x2="50.8" y2="30.48" width="0.1524" layer="91"/>
-<junction x="50.8" y="30.48"/>
-<wire x1="50.8" y1="30.48" x2="106.68" y2="30.48" width="0.1524" layer="91"/>
-<wire x1="106.68" y1="30.48" x2="106.68" y2="60.96" width="0.1524" layer="91"/>
-<wire x1="106.68" y1="60.96" x2="106.68" y2="66.04" width="0.1524" layer="91"/>
-<wire x1="101.6" y1="66.04" x2="106.68" y2="66.04" width="0.1524" layer="91"/>
-<wire x1="101.6" y1="60.96" x2="106.68" y2="60.96" width="0.1524" layer="91"/>
-<junction x="106.68" y="60.96"/>
-<pinref part="U$1" gate="G$1" pin="GND@1"/>
-<pinref part="U$1" gate="G$1" pin="GND@2"/>
-<wire x1="27.94" y1="55.88" x2="30.48" y2="55.88" width="0.1524" layer="91"/>
-<wire x1="30.48" y1="55.88" x2="30.48" y2="30.48" width="0.1524" layer="91"/>
-<pinref part="X1" gate="-2" pin="KL"/>
+<wire x1="68.58" y1="73.66" x2="68.58" y2="78.74" width="0.1524" layer="91"/>
 </segment>
 </net>
